File: NanoCore-525/NanoCore-525.kicad_sch (KiCad schematic)
At the start: 22 parts, among them J1 Conn_01x02, J2 Conn_01x02, J3 Conn_01x02, J4 Conn_01x02, J5 Conn_01x02, J6 Conn_01x02, SW1 SW_Push

Commit message: update
Parts:
- added TP3: TestPoint, TestPoint:TestPoint_Pad_D1.0mm, symbol Connector:TestPoint
- added Vout6: -, B2PS-VH:JST_VH_B2PS-VH_1x02_P3.96mm_Horizontal, symbol Connector_Generic:Conn_01x02
- C_IN1, C_IN2: Mfr. No (none) -> UMK325AB7106MM-T; Mouser No (none) -> 963-UMK325AB7106MM-T
- C_OUT1, C_OUT2: Mfr. No (none) -> CL32B476KPJNNNE; Mouser No (none) -> 187-CL32B476KPJNNNE
- NT1, NT2: footprint (none) -> NetTie:NetTie-2_SMD_Pad2.0mm
- R_ENB1: renamed from R_ENB; footprint (none) -> Resistor_SMD:R_0402_1005Metric_Pad0.72x0.64mm_HandSolder
- R_ENT1: renamed from R_ENT; footprint (none) -> Resistor_SMD:R_0402_1005Metric_Pad0.72x0.64mm_HandSolder
- R_FBB1: renamed from R_FBB; footprint (none) -> Resistor_SMD:R_0402_1005Metric_Pad0.72x0.64mm_HandSolder
- R_FBT1: renamed from R_FBT; footprint (none) -> Resistor_SMD:R_0402_1005Metric_Pad0.72x0.64mm_HandSolder
- R_RT1: renamed from R_RT; footprint (none) -> Resistor_SMD:R_0402_1005Metric_Pad0.72x0.64mm_HandSolder
- TP1, TP2: footprint (none) -> TestPoint:TestPoint_Pad_D1.0mm
- U3: footprint Package_DFN_QFN:Texas_B3QFN-14-1EP_5x5.5mm_P0.65mm_ThermalVia -> TLVM:B3QFN20_RDL_TEX; Mfr. No (none) -> TLVM13660RDLR; Mouser No (none) -> 595-TLVM13660RDLR
- VIN1: renamed from J6; value Conn_01x02 -> -; footprint (none) -> Connector_JST:JST_VH_B2P-VH-B_1x02_P3.96mm_Vertical; Mfr. No (none) -> B2P-VH-B(LF)(SN); Mouser No (none) -> 306-306-B2PVHBLFSN
- Vout1: renamed from J1; value Conn_01x02 -> -; footprint (none) -> B2PS-VH:JST_VH_B2PS-VH_1x02_P3.96mm_Horizontal; Mfr. No (none) -> B2PS-VH(LF)(SN); Mouser No (none) -> 306-B2PS-VHLFSN
- Vout2: renamed from J2; value Conn_01x02 -> -; footprint (none) -> B2PS-VH:JST_VH_B2PS-VH_1x02_P3.96mm_Horizontal; Mfr. No (none) -> B2PS-VH(LF)(SN); Mouser No (none) -> 306-B2PS-VHLFSN
- Vout3: renamed from J3; value Conn_01x02 -> -; footprint (none) -> B2PS-VH:JST_VH_B2PS-VH_1x02_P3.96mm_Horizontal; Mfr. No (none) -> B2PS-VH(LF)(SN); Mouser No (none) -> 306-B2PS-VHLFSN
- Vout4: renamed from J4; value Conn_01x02 -> -; footprint (none) -> B2PS-VH:JST_VH_B2PS-VH_1x02_P3.96mm_Horizontal; Mfr. No (none) -> B2PS-VH(LF)(SN); Mouser No (none) -> 306-B2PS-VHLFSN
- Vout5: renamed from J5; value Conn_01x02 -> -; footprint (none) -> B2PS-VH:JST_VH_B2PS-VH_1x02_P3.96mm_Horizontal; Mfr. No (none) -> B2PS-VH(LF)(SN); Mouser No (none) -> 306-B2PS-VHLFSN
- renumbered C_FF to C_FF1
Connections:
- net GND is gone; now on net PGND: Vout1.1 (Pin_1), Vout2.1 (Pin_1), Vout3.1 (Pin_1), Vout4.1 (Pin_1), Vout5.1 (Pin_1)
- net +5V: now also Vout6.2 (Pin_2)
- net PGND: now also TP3.1, Vout6.1 (Pin_1)
- net SW_EN: now reaches R_ENT1.1, SW1.1
- net FB: now reaches C_FF1.2, R_FBB1.1, R_FBT1.2, U3.10 (FB)
- net RT: now reaches R_RT1.1, U3.12 (RT)
- net RBOOT: now reaches U3.3 (CBOOT), U3.4 (RBOOT)
Other:
- moved on the sheet: SW1, Vout1, Vout2, Vout3, Vout4, Vout5
